File: hardware/sss7modem.kicad_pcb (KiCad board)
At the start: 2 copper layers, 34.3 x 44.4 mm, 37 parts, among them IC1 MCP2551-I/SN, IC2 LTV-352T, IC3 LTV-352T, K1 CONN_3, P1 CONN_4, U1 SIM1-0505, U2 74HCT125

Commit message: Finalized pcb layout and silkscreen
Parts:
- IC1: value MCP2551-I/SN -> MCP2551
- moved G*** 1.91 mm to (40.6, 44.5)
- moved G*** 0.64 mm to (48.3, 61.0)
Other:
- board text added: "+5v"
- board text added: "BUS GND"
- board text added: "BUS H"
- board text added: "BUS L"
- board text added: "GND"
- board text added: "RXD/OUT"
- board text added: "SSS7 Modem"
- board text added: "TXD/IN"
- board text added: "Version 1.0 by Sebastian Schumb 2015"
- board text added: "https://github.com/seidenstrasse/sss7modem"
Changed lines of the file:
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@@
     (area 10.415002 16.200001 57.835001 79.535)
     (thickness 1.6)
-    (drawings 17)
+    (drawings 28)
     (tracks 131)
     (zones 0)
@@
   (page A3)
   (layers
-    (15 F.Cu signal hide)
-    (0 B.Cu signal hide)
+    (15 F.Cu signal)
+    (0 B.Cu signal)
     (16 B.Adhes user)
     (17 F.Adhes user)
     (18 B.Paste user)
     (19 F.Paste user)
-    (20 B.SilkS user hide)
+    (20 B.SilkS user)
     (21 F.SilkS user)
     (22 B.Mask user)
@@
     (tags "CMS SOJ")
     (attr smd)
-    (fp_text reference IC1 (at 0 -0.889) (layer F.SilkS)
-      (effects (font (size 1.143 1.143) (thickness 0.1524)))
+    (fp_text reference IC1 (at 3.81 -1.27) (layer F.SilkS)
+      (effects (font (size 0.75 0.75) (thickness 0.2)))
     )
-    (fp_text value MCP2551-I/SN (at 0 1.016) (layer F.SilkS)
-      (effects (font (size 0.889 0.889) (thickness 0.1524)))
+    (fp_text value MCP2551 (at 0 1.27) (layer F.SilkS)
+      (effects (font (size 0.75 0.75) (thickness 0.1875)))
     )
     (fp_line (start -2.667 1.778) (end -2.667 1.905) (layer F.SilkS) (width 0.127))
@@
     (at 48.895 57.785)
     (attr smd)
-    (fp_text reference C2 (at 0 0) (layer F.SilkS)
-      (effects (font (size 0.508 0.4572) (thickness 0.1143)))
+    (fp_text reference C2 (at -1.905 1.27) (layer F.SilkS)
+      (effects (font (size 0.75 0.75) (thickness 0.2)))
     )
     (fp_text value 100nF (at 0 0) (layer F.SilkS) hide
@@
     (at 51.435 62.23)
     (descr "SMT capacitor, aluminium electrolytic, 6.3x5.8")
-    (fp_text reference C1 (at 0 -3.937) (layer F.SilkS)
-      (effects (font (size 0.50038 0.50038) (thickness 0.11938)))
+    (fp_text reference C1 (at 0.635 4.445) (layer F.SilkS)
+      (effects (font (size 0.75 0.75) (thickness 0.2)))
     )
     (fp_text value 47uF (at 0 3.81) (layer F.SilkS) hide
@@
     (descr "Bornier d'alimentation 4 pins")
     (tags DEV)
-    (fp_text reference P1 (at 0 -6.35) (layer F.SilkS)
-      (effects (font (size 2.6162 1.59766) (thickness 0.3048)))
+    (fp_text reference P1 (at -9.525 -5.08) (layer F.SilkS)
+      (effects (font (size 0.75 0.75) (thickness 0.2)))
     )
     (fp_text value CONN_4 (at 0 5.08) (layer F.SilkS) hide
@@
     (at 46.99 46.355 270)
     (attr smd)
-    (fp_text reference R8 (at 0 0 360) (layer F.SilkS)
-      (effects (font (size 0.508 0.4572) (thickness 0.1143)))
+    (fp_text reference R8 (at 0 1.905 360) (layer F.SilkS)
+      (effects (font (size 0.75 0.75) (thickness 0.2)))
     )
     (fp_text value 390 (at 0 0 270) (layer F.SilkS) hide
@@
     (at 48.895 55.245 270)
     (attr smd)
-    (fp_text reference R7 (at 0 0 270) (layer F.SilkS)
-      (effects (font (size 0.508 0.4572) (thickness 0.1143)))
+    (fp_text reference R7 (at -1.905 0 360) (layer F.SilkS)
+      (effects (font (size 0.75 0.75) (thickness 0.2)))
     )
     (fp_text value R (at 0 0 270) (layer F.SilkS) hide
@@
     (at 55.245 46.355)
     (attr smd)
-    (fp_text reference C4 (at 0 0) (layer F.SilkS)
-      (effects (font (size 0.508 0.4572) (thickness 0.1143)))
+    (fp_text reference C4 (at 0 1.905) (layer F.SilkS)
+      (effects (font (size 0.75 0.75) (thickness 0.2)))
     )
     (fp_text value 100nF (at 0 0) (layer F.SilkS) hide
@@
     (descr "Connecteur 4 pibs")
     (tags "CONN DEV")
-    (fp_text reference U1 (at 0 -2.54 90) (layer F.SilkS)
-      (effects (font (size 1.73482 1.08712) (thickness 0.3048)))
+    (fp_text reference U1 (at -5.08 2.54 180) (layer F.SilkS)
+      (effects (font (size 0.75 0.75) (thickness 0.2)))
     )
     (fp_text value SIM1-0505 (at 0 -2.54 90) (layer F.SilkS) hide
@@
     (at 52.07 41.275 270)
     (descr "SMT capacitor, aluminium electrolytic, 6.3x5.8")
-    (fp_text reference C3 (at 3.81 3.175 360) (layer F.SilkS)
+    (fp_text reference C3 (at 0 -4.445 360) (layer F.SilkS)
       (effects (font (size 0.75 0.75) (thickness 0.2)))
     )
@@
     (tags "CMS SOJ")
     (attr smd)
-    (fp_text reference U2 (at 0 -0.762) (layer F.SilkS)
-      (effects (font (size 1.016 1.143) (thickness 0.127)))
+    (fp_text reference U2 (at -5.715 2.54) (layer F.SilkS)
+      (effects (font (size 0.75 0.75) (thickness 0.2)))
     )
-    (fp_text value 74HCT125 (at 0 1.016) (layer F.SilkS)
-      (effects (font (size 1.016 1.016) (thickness 0.127)))
+    (fp_text value 74HCT125 (at 0 -0.635) (layer F.SilkS)
+      (effects (font (size 0.75 0.75) (thickness 0.2)))
     )
     (fp_line (start -4.826 -1.778) (end 4.826 -1.778) (layer F.SilkS) (width 0.2032))
@@
     (at 39.37 52.705)
     (descr "Mini flat package, 4 pin")
-    (fp_text reference IC3 (at 0 -5) (layer F.SilkS)
-      (effects (font (size 1 1) (thickness 0.2)))
+    (fp_text reference IC3 (at 3.175 -1.27) (layer F.SilkS)
+      (effects (font (size 0.75 0.75) (thickness 0.2)))
     )
     (fp_text value LTV-352T (at 0 5.1) (layer F.SilkS) hide
@@
     (at 45.72 52.705 180)
     (descr "Mini flat package, 4 pin")
-    (fp_text reference IC2 (at 0 -5 180) (layer F.SilkS)
-      (effects (font (size 1 1) (thickness 0.2)))
+    (fp_text reference IC2 (at -3.175 1.27 180) (layer F.SilkS)
+      (effects (font (size 0.75 0.75) (thickness 0.2)))
     )
-    (fp_text value LTV-352T (at 0 5.1 180) (layer F.SilkS)
+    (fp_text value LTV-352T (at 0 5.1 180) (layer F.SilkS) hide
       (effects (font (size 1 1) (thickness 0.2)))
     )
@@
   )
   (module seidenstrasse_silkbot_15_00mm (layer B.Cu)
-    (at 40.64 42.545)
+    (at 40.64 44.45)
     (fp_text reference G*** (at 0 -7.66064) (layer B.SilkS) hide
       (effects (font (size 0.26416 0.26416) (thickness 0.0508)) (justify mirror))
@@
   )
   (module chaosinkl_silkbot_15_00mm (layer B.Cu)
-    (at 48.895 60.96)
+    (at 48.26 60.96)
     (fp_text reference G*** (at 0 -5.58546) (layer B.SilkS) hide
       (effects (font (size 0.29972 0.29972) (thickness 0.05842)) (justify mirror))
@@
       (xy -0.14224 -2.76098) (xy -0.14224 -2.75336) (xy -0.14224 -2.74066) (xy -0.14224 -2.74066)) (layer B.SilkS) (width 0.00254))
   )
-  (gr_line (start 24.13 52.705) (end 57.15 52.705) (angle 90) (layer B.SilkS) (width 0.2))
+  (gr_line (start 24.13 52.705) (end 55.88 52.705) (angle 90) (layer B.SilkS) (width 0.2))
+  (gr_text "BUS L" (at 40.64 35.56) (layer B.SilkS)
+    (effects (font (size 0.75 0.75) (thickness 0.1875)) (justify mirror))
+  )
+  (gr_text "BUS H" (at 35.56 35.56) (layer B.SilkS)
+    (effects (font (size 0.75 0.75) (thickness 0.1875)) (justify mirror))
+  )
+  (gr_text "BUS GND" (at 45.72 35.56) (layer B.SilkS)
+    (effects (font (size 0.75 0.75) (thickness 0.1875)) (justify mirror))
+  )
+  (gr_text GND (at 33.02 66.675) (layer B.SilkS)
+    (effects (font (size 0.75 0.75) (thickness 0.1875)) (justify mirror))
+  )
+  (gr_text +5v (at 48.26 66.675) (layer B.SilkS)
+    (effects (font (size 0.75 0.75) (thickness 0.1875)) (justify mirror))
+  )
+  (gr_text RXD/OUT (at 43.18 66.675) (layer B.SilkS)
+    (effects (font (size 0.75 0.75) (thickness 0.1875)) (justify mirror))
+  )
+  (gr_text TXD/IN (at 38.1 66.675) (layer B.SilkS)
+    (effects (font (size 0.75 0.75) (thickness 0.1875)) (justify mirror))
+  )
+  (gr_text "SSS7 Modem" (at 25.4 43.18 90) (layer F.SilkS)
+    (effects (font (size 1.5 1.5) (thickness 0.375)))
+  )
+  (gr_text https://github.com/seidenstrasse/sss7modem (at 56.515 36.195 90) (layer B.SilkS)
+    (effects (font (size 0.75 0.75) (thickness 0.1875)) (justify left mirror))
+  )
+  (gr_text "Version 1.0\nby Sebastian Schumb 2015\n" (at 53.34 36.195 90) (layer B.SilkS)
+    (effects (font (size 0.75 0.75) (thickness 0.1875)) (justify left mirror))
+  )
+  (gr_text "SSS7 Modem" (at 25.4 43.18 90) (layer B.SilkS)
+    (effects (font (size 1.5 1.5) (thickness 0.375)) (justify mirror))
+  )
   (dimension 34.29 (width 0.3) (layer Cmts.User)
     (gr_text "34.290 mm" (at 40.64 78.184999) (layer Cmts.User)
